File: boards/pico-controller/pico-controller.kicad_pcb (KiCad board)
At the start: 2 copper layers, 130 x 80 mm, 125 parts, among them J1 Conn_01x02_Male, J10 Conn_01x03_Male, J11 Conn_01x03_Male, J12 Conn_01x03_Male, J13 Conn_01x03_Male, J14 Conn_01x03_Male, J15 Conn_01x03_Male, J16 Conn_01x02_Male, J17 Conn_01x02_Male, J18 Conn_01x02_Male, J19 Conn_01x02_Male, J20 Conn_01x02_Male, J21 Conn_01x06_Male, J22 LCD I2C, J23 Conn_01x07_Male, J3 Conn_01x02_Male, J8 Conn_01x04_Male, J9 Conn_01x04_Male, Q1 BSS138, Q10 BSS138, Q11 BSS138, Q12 BSS138, Q13 BSS138, Q14 TIP122, Q15 BSS138, Q16 BSS138, Q17 BC817, Q18 BC817, Q2 BSS138, Q3 BSS138, Q4 BSS138, Q5 BSS138, Q6 BSS138, Q7 BSS138, Q8 BSS138, Q9 BSS138, SW1 SW_Push, U1 MCP3208, U2 LM4040DBZ-5.0, U3 24LC1025, U4 Pico, U5 IR2110, U6 IR2110

Commit message: pico-controller: switched to kicad 7
Connections:
- net /HV_MCP_~CS~ renamed /HV_MCP_~{CS}
- net /SPI_PICO_~CS~ renamed /SPI_PICO_~{CS}
- net /~RESET~ renamed /~{RESET}
Other:
- net class Default removed
- net class H-Driver removed
- net class Power removed
