File: boards/power-driver/power-driver.kicad_pcb (KiCad board)
At the start: 2 copper layers, 53.3 x 50.8 mm, 36 parts, among them J1 Conn_01x02_Female, J2 Conn_01x06_Male, J3 Conn_01x04_Male, U1 L7805, U2 6N137, U3 6N137, U4 6N137, U5 IR2110

Commit message: power-driver: updated to kicad 7
Other:
- net class Default removed
